Commit message: Cone detection setup with OpenCV and YOLO

File: src/4wd_robot_sim/urdf/4wd_robot.xacro (robot description, xacro)
@@ -92,4 +92,14 @@
       <material name="black"/>
     </visual>
+    <collision>
+      <geometry>
+        <box size="0.05 0.05 0.05"/>
+      </geometry>
+      <origin xyz="0 0 0" rpy="0 0 0"/>
+    </collision>
+    <inertial>
+      <mass value="0.1"/>
+      <inertia ixx="0.0001" iyy="0.0001" izz="0.0001" ixy="0" ixz="0" iyz="0"/>
+    </inertial>
   </link>
   <joint name="camera_joint" type="fixed">
@@ -100,9 +110,9 @@
   <gazebo reference="camera_link">
     <sensor name="camera_sensor" type="camera">
+      <update_rate>30.0</update_rate>
       <always_on>true</always_on>
-      <update_rate>30.0</update_rate>
       <visualize>true</visualize>
       <camera>
-        <horizontal_fov>1.047</horizontal_fov>
+        <horizontal_fov>1.3962634</horizontal_fov>
         <image>
           <width>640</width>
@@ -116,8 +126,7 @@
       </camera>
       <plugin name="gazebo_ros_camera" filename="libgazebo_ros_camera.so">
-        <ros>
-          <remapping>~/image_raw:=/camera/image_raw</remapping>
-        </ros>
         <camera_name>camera</camera_name>
+        <image_topic_name>image_raw</image_topic_name>
+        <camera_info_topic_name>camera_info</camera_info_topic_name>
         <frame_name>camera_link</frame_name>
       </plugin>
@@ -169,11 +178,9 @@
     </inertial>
   </link>
-  <joint name="lidar_joint" type="continuous">
+  <joint name="lidar_joint" type="fixed">
     <parent link="lidar_stand_link"/>
     <child link="lidar_link"/>
     <origin xyz="0 0 0.4" rpy="0 0 0"/>
-    <axis xyz="0 0 1"/>
   </joint>
-  <!-- ✅ 360° LIDAR Configuration -->
   <gazebo reference="lidar_link">
     <sensor name="rotating_lidar" type="ray">
@@ -184,8 +191,8 @@
         <scan>
           <horizontal>
-            <samples>720</samples>
+            <samples>360</samples>
             <resolution>1</resolution>
-            <min_angle>-3.14</min_angle>
-            <max_angle>3.14</max_angle>
+            <min_angle>-1.57</min_angle>
+            <max_angle>1.57</max_angle>
           </horizontal>
         </scan>
@@ -205,5 +212,5 @@
     </sensor>
   </gazebo>
-  <!-- Diff Drive Plugin (front wheels only) -->
+  <!-- Diff Drive -->
   <gazebo>
     <plugin name="diff_drive" filename="libgazebo_ros_diff_drive.so">
